File: STM32F411 Circuitry.kicad_sch (KiCad schematic)
At the start: 28 parts, among them J3 USB_C_Receptacle_USB2.0_16P, J8 Conn_01x04_Pin, J9 Conn_01x02_Pin, SW1 SW_Push, SW2 SW_Push, U1 STM32F411CEUx, U4 TLV70233_SOT23-5, Y1 Crystal_GND23, Y2 Crystal

Commit message: new pcb. added power switch and disc detect button
rfid reading has been unreliable, so added a button that gets pressed when a disc is inserted to lock the current disc that's playing. eliminates the chance of a music disc that's inserted to randomly stop playing due to the rfid reader's wonky detection not catching its presence
Parts:
- added J10: Conn_1x1, TestPoint:TestPoint_THTPad_D1.0mm_Drill0.5mm, symbol Connector:Conn_01x01_Socket
- added SW3: SW_SPST, Connector_PinHeader_2.00mm:PinHeader_1x02_P2.00mm_Vertical, symbol Switch:SW_SPST
Connections:
- net +5V: now also SW3.2 (B); no longer J3.A4 (VBUS), J3.A9 (VBUS), J3.B4 (VBUS), J3.B9 (VBUS)
- net Insert_Disc_Detect: now reaches U1.11 (PA1)
- net Insert_Disc_Detect: now also J10.1 (Pin_1)
- new net USB_5V: J3.A4 (VBUS), J3.A9 (VBUS), J3.B4 (VBUS), J3.B9 (VBUS), SW3.1 (A)
- no-connect marks 7 -> 6
Other:
- moved on the sheet: R17, R18
